Commit message: Created basic transforms for vision visualization

File: aidu_vision/urdf/base.urdf (robot description, URDF)
Before this commit: robot aidu, 1 links, 0 joints
Links:
- added link camera_link
- added link main_link; visual box size=0.57 0.46 0.08
- link base_link: geometry 
Joints:
- added joint base_camera: type fixed, parent base_link, child camera_link, origin xyz=0.06 0 0.23
- added joint base_main: type fixed, parent base_link, child main_link, origin xyz=-0.201 0 0.14
