Commit message: Calibrated camera positioning on base in our urdf model

File: aidu_transforms/urdf/base.urdf (robot description, URDF)
Before this commit: robot aidu, 3 links, 2 joints
Joints:
- joint base_camera: origin xyz=0.06 0 0.23 -> xyz=0.077 0 0.228

Commit message: Modified position of kinect

File: aidu_transforms/urdf/base.urdf (robot description, URDF)
Before this commit: robot aidu, 3 links, 2 joints
Joints:
- joint base_camera: origin xyz=0.077 0 0.228 -> xyz=-0.32 0 0.40

Commit message: changed position of kinect

File: aidu_transforms/urdf/base.urdf (robot description, URDF)
Before this commit: robot aidu, 3 links, 2 joints
Joints:
- joint base_camera: origin xyz=-0.32 0 0.40 -> xyz=0 0 0.23

Commit message: added robot arm links and joints

File: aidu_transforms/urdf/base.urdf (robot description, URDF)
Before this commit: robot aidu, 3 links, 2 joints
Links:
- added link rotationalarm_link; visual box size=0.135 0.015 0.015
- added link spindlecaddy_link; visual box size=0.08 0.065 0.0467
- added link webcam_link; visual box size=0.02 0.045 0.037
Joints:
- added joint base_spindlecaddy: type prismatic, parent base_link, child spindlecaddy_link, origin xyz=0.1 -0.2 0.7, axis 0 0 1, limit lower=0 upper=0.5 effort=1000.0 velocity=0.7
- added joint rotationalarm_webcam: type fixed, parent rotationalarm_link, child webcam_link, origin xyz=0.03 0 0.026
- added joint spindlecaddy_rotationalarm: type revolute, parent spindlecaddy_link, child rotationalarm_link, origin xyz=0.0925 0.0 0.0413, axis 0 0 1, limit lower=0 upper=0.5 effort=1000.0 velocity=0.7

Commit message: added robot_arm to urdf

File: aidu_transforms/urdf/base.urdf (robot description, URDF)
Before this commit: robot aidu, 6 links, 5 joints
Links:
- added link extension_link; visual box size=0.10 0.009 0.009
Joints:
- added joint rotationalarm_extension: type prismatic, parent rotationalarm_link, child extension_link, origin xyz=0.04 -0.001 0.0, axis 1 0 0, limit lower=0 upper=0.10 effort=1000.0 velocity=0.3
- joint spindlecaddy_rotationalarm: limit lower=0 upper=0.5 effort=1000.0 velocity=0.7 -> lower=0 upper=3.1415 effort=1000.0 velocity=3.1415

Commit message: implemented joint state publsiher

File: aidu_transforms/urdf/base.urdf (robot description, URDF)
Before this commit: robot aidu, 7 links, 6 joints
Links:
- link extension_link: geometry visual box size=0.14 0.009 0.009
- link rotationalarm_link: geometry visual box size=0.15 0.015 0.015
Joints:
- joint rotationalarm_extension: limit lower=0 upper=0.10 effort=1000.0 velocity=0.3 -> lower=0 upper=0.075 effort=1000.0 velocity=0.3; origin xyz=0.04 -0.001 0.0 -> xyz=0.150 -0.001 0.0075
- joint rotationalarm_webcam: origin xyz=0.03 0 0.026 -> xyz=0.03 0 0.0335
- joint spindlecaddy_rotationalarm: limit lower=0 upper=3.1415 effort=1000.0 velocity=3.1415 -> lower=-1.57 upper=1.57 effort=1000.0 velocity=3.1415; origin xyz=0.0925 0.0 0.0413 -> xyz=0.0 0.0 0.01

Commit message: created robot model

File: aidu_transforms/urdf/base.urdf (robot description, URDF)
Before this commit: robot aidu, 7 links, 6 joints
Links:
- added link kast_link; visual mesh filename=package://aidu_transforms/urdf/kast2.STL scale=0.001 0.001 0.001
- added link kinect_link; visual mesh filename=package://aidu_transforms/urdf/Kinect.STL scale=0.001 0.001 0.001
- added link lade1_link; visual mesh filename=package://aidu_transforms/urdf/lade1.STL scale=0.001 0.001 0.001
- added link lade2_link; visual mesh filename=package://aidu_transforms/urdf/lade2.STL scale=0.001 0.001 0.001
- added link lade3_link; visual mesh filename=package://aidu_transforms/urdf/lade3.STL scale=0.001 0.001 0.001
- added link macbook_link; visual mesh filename=package://aidu_transforms/urdf/MacBook.STL scale=0.001 0.001 0.001
Joints:
- added joint main_kast: type fixed, parent main_link, child kast_link, origin xyz=0.285 -0.23 1.2
- added joint main_kinect: type fixed, parent main_link, child kinect_link, origin xyz=0.235 -0.14 0.05
- added joint main_lade1: type fixed, parent main_link, child lade1_link, origin xyz=-0.225 0.185 0.0
- added joint main_lade2: type fixed, parent main_link, child lade2_link, origin xyz=-0.225 0.185 0.445
- added joint main_lade3: type fixed, parent main_link, child lade3_link, origin xyz=-0.225 0.185 0.75
- added joint main_macbook: type fixed, parent main_link, child macbook_link, origin xyz=0.1 0.21 1.18

Commit message: navigation parameters

File: aidu_transforms/urdf/base.urdf (robot description, URDF)
Before this commit: robot aidu, 13 links, 12 joints
Links:
- removed link extension_link
- removed link kast_link
- removed link kinect_link
- removed link lade1_link
- removed link lade2_link
- removed link lade3_link
- removed link macbook_link
- removed link rotationalarm_link
- removed link spindlecaddy_link
- removed link webcam_link
Joints:
- removed joint base_spindlecaddy
- removed joint main_kast
- removed joint main_kinect
- removed joint main_lade1
- removed joint main_lade2
- removed joint main_lade3
- removed joint main_macbook
- removed joint rotationalarm_extension
- removed joint rotationalarm_webcam
- removed joint spindlecaddy_rotationalarm

Commit message: other stuff

File: aidu_transforms/urdf/base.urdf (robot description, URDF)
Before this commit: robot aidu, 3 links, 2 joints
Links:
- added link extension_link; visual box size=0.14 0.009 0.009
- added link rotationalarm_link; visual box size=0.15 0.015 0.015
- added link spindlecaddy_link; visual box size=0.08 0.065 0.0467
- added link webcam_link; visual box size=0.02 0.045 0.037
Joints:
- added joint base_spindlecaddy: type prismatic, parent base_link, child spindlecaddy_link, origin xyz=0.108 -0.1525 0.905, axis 0 0 1, limit lower=0 upper=0.5 effort=1000.0 velocity=0.7
- added joint rotationalarm_extension: type prismatic, parent rotationalarm_link, child extension_link, origin xyz=0.150 -0.001 0.0075, axis 1 0 0, limit lower=0 upper=0.075 effort=1000.0 velocity=0.3
- added joint rotationalarm_webcam: type fixed, parent rotationalarm_link, child webcam_link, origin xyz=0.03 0 0.0335
- added joint spindlecaddy_rotationalarm: type revolute, parent spindlecaddy_link, child rotationalarm_link, origin xyz=0.0 0.0 0.01, axis 0 0 1, limit lower=-1.57 upper=1.57 effort=1000.0 velocity=3.1415
